File: ft2232breakout.sch (KiCad schematic (older format))
At the start: 24 parts, among them J1 USB_B_Micro, J2 Conn_01x20, J3 Conn_01x20, U1 FT2232H, U2 NCP1117-3.3_SOT223, U3 93CxxA

Commit message: Nearly there
Parts:
- removed U3: 93CxxA, Package_SO:SOIC-8_3.9x4.9mm_P1.27mm, symbol Memory_EEPROM:93CxxA
- added C15, C16: 27pF, Capacitor_SMD:C_0603_1608Metric_Pad1.05x0.95mm_HandSolder, symbol Device:C
- added C17: 4.7uF, Capacitor_SMD:C_0603_1608Metric_Pad1.05x0.95mm_HandSolder, symbol Device:C
- added R1: 12k, Resistor_SMD:R_0603_1608Metric_Pad1.05x0.95mm_HandSolder, symbol Device:R
- added R2: 1k, Resistor_SMD:R_0603_1608Metric_Pad1.05x0.95mm_HandSolder, symbol Device:R
- added R3: 2.2k, Resistor_SMD:R_0603_1608Metric_Pad1.05x0.95mm_HandSolder, symbol Device:R
- added R4, R5, R6: 10k, Resistor_SMD:R_0603_1608Metric_Pad1.05x0.95mm_HandSolder, symbol Device:R
- added U3: 93LCxxAxxOT, Package_TO_SOT_SMD:SOT-23-6, symbol Memory_EEPROM:93LCxxAxxOT
- added Y1: 12MHz, Crystal:Crystal_SMD_3225-4Pin_3.2x2.5mm_HandSoldering, symbol Device:Crystal_GND24
- C1, C10, C11, C12, C13, C14, C2, C4, C7, C8, C9: Digikey (none) -> 1276-1000-1-ND; Digikey Link (none) -> https://www.digikey.com/product-detail/en/samsung-electro-m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
- C3, C5, C6: Digikey (none) -> 1276-6684-1-ND; Digikey Link (none) -> https://www.digikey.com/product-detail/en/samsung-electro-m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
- J1: Digikey (none) -> WM1399CT-ND; Digikey Link (none) -> https://www.digikey.com/product-detail/en/molex/1050170001/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
- U2: value NCP1117-3.3_SOT223 -> NCP1117ST33T3G
Connections:
- net +3V3: now also J2.1 (Pin_1), J3.1 (Pin_1), C17.1, R2.2, R4.2, R5.2, R6.2, U3.6 (VCC)
- net GND: now also J2.2 (Pin_2), J2.20 (Pin_20), J3.2 (Pin_2), J3.20 (Pin_20), U1.1 (GND), U1.10 (AGND), U1.11 (GND), U1.13 (TEST), U1.15 (GND), U1.25 (GND), U1.35 (GND), U1.47 (GND), U1.5 (GND), U1.51 (GND), C15.2, C16.2, C17.2, R1.2, U3.2 (GND), Y1.2, Y1.4
- net at U1.14 (~RESET): now also R2.1
- net AD0: now reaches J2.3 (Pin_3), U1.16 (ADBUS0)
- net AD1: now reaches J2.4 (Pin_4), U1.17 (ADBUS1)
- net AD2: now reaches J2.5 (Pin_5), U1.18 (ADBUS2)
- net AD3: now reaches J2.6 (Pin_6), U1.19 (ADBUS3)
- net at U1.2 (OSCI): now also C15.1, Y1.1
- net AD4: now reaches J2.7 (Pin_7), U1.21 (ADBUS4)
- net AD5: now reaches J2.8 (Pin_8), U1.22 (ADBUS5)
- net AD6: now reaches J2.9 (Pin_9), U1.23 (ADBUS6)
- net AD7: now reaches J2.10 (Pin_10), U1.24 (ADBUS7)
- net AC0: now reaches J2.11 (Pin_11), U1.26 (ACBUS0)
- net AC1: now reaches J2.12 (Pin_12), U1.27 (ACBUS1)
- net AC2: now reaches J2.13 (Pin_13), U1.28 (ACBUS2)
- net AC3: now reaches J2.14 (Pin_14), U1.29 (ACBUS3)
- net at U1.3 (OSCO): now also C16.1, Y1.3
- net AC4: now reaches J2.15 (Pin_15), U1.30 (ACBUS4)
- net AC5: now reaches J2.16 (Pin_16), U1.32 (ACBUS5)
- net AC6: now reaches J2.17 (Pin_17), U1.33 (ACBUS6)
- net AC7: now reaches J2.18 (Pin_18), U1.34 (ACBUS7)
- net ~SUSPEND: now reaches U1.36 (~SUSPEND)
- net ~SUSPEND: now also J2.19 (Pin_19)
- net BD0: now reaches J3.3 (Pin_3), U1.38 (BDBUS0)
- net BD1: now reaches J3.4 (Pin_4), U1.39 (BDBUS1)
- net BD2: now reaches J3.5 (Pin_5), U1.40 (BDBUS2)
- net BD3: now reaches J3.6 (Pin_6), U1.41 (BDBUS3)
- net BD4: now reaches J3.7 (Pin_7), U1.43 (BDBUS4)
- net BD5: now reaches J3.8 (Pin_8), U1.44 (BDBUS5)
- net BD6: now reaches J3.9 (Pin_9), U1.45 (BDBUS6)
- net BD7: now reaches J3.10 (Pin_10), U1.46 (BDBUS7)
- net BC0: now reaches J3.11 (Pin_11), U1.48 (BCBUS0)
- net BC1: now reaches J3.12 (Pin_12), U1.52 (BCBUS1)
- net BC2: now reaches J3.13 (Pin_13), U1.53 (BCBUS2)
- net BC3: now reaches J3.14 (Pin_14), U1.54 (BCBUS3)
- net BC4: now reaches J3.15 (Pin_15), U1.55 (BCBUS4)
- net BC5: now reaches J3.16 (Pin_16), U1.57 (BCBUS5)
- net BC6: now reaches J3.17 (Pin_17), U1.58 (BCBUS6)
- net BC7: now reaches J3.18 (Pin_18), U1.59 (BCBUS7)
- net at U1.6 (REF): now also R1.1
- net ~PWREN: now reaches U1.60 (~PWREN)
- net ~PWREN: now also J3.19 (Pin_19)
- net at U1.61 (EEDATA): now also R3.2, R4.1, U3.3 (DI)
- net at U1.62 (EECLK): now also R5.1, U3.4 (CLK)
- net at U1.63 (EECS): now also R6.1, U3.5 (CS)
- new net: R3.1, U3.1 (DO)
Other:
- moved on the sheet: C3, C4, C6, C7

Commit message: Made board smaller
Parts:
- C1, C10, C11, C12, C13, C14, C15, C16, C17, C2, C3, C4, C5, C6, C7, C8, C9: footprint Capacitor_SMD:C_0603_1608Metric_Pad1.05x0.95mm_HandSolder -> Capacitor_SMD:C_0603_1608Metric
- R1, R2, R3, R4, R5, R6: footprint Resistor_SMD:R_0603_1608Metric_Pad1.05x0.95mm_HandSolder -> Resistor_SMD:R_0603_1608Metric
- U1: Digikey (none) -> 768-1024-2-ND; Digikey URL (none) -> https://www.digikey.my/product-detail/en/ftdi-future-techno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
Changed lines of the file:
@@
 EESchema Schematic File Version 4
 LIBS:ft2232breakout-cache
-EELAYER 29 0
+EELAYER 30 0
 EELAYER END
 $Descr A4 11693 8268
@@
 F 2 "Package_QFP:LQFP-64_10x10mm_P0.5mm" H 5700 4400 50  0001 C CNN
 F 3 "http://www.ftdichip.com/Products/ICs/FT2232H.html" H 5700 4400 50  0001 C CNN
+F 4 "768-1024-2-ND" H 5700 4400 50  0001 C CNN "Digikey"
+F 5 "https://www.digikey.my/product-detail/en/ftdi-future-technology-devices-international-ltd/FT2232HL-REEL/768-1024-2-ND/1986053" H 5700 4400 50  0001 C CNN "Digikey URL"
 	1    5700 4400
 	1    0    0    -1
@@
 F 0 "C2" H 2015 1996 50  0000 L CNN
 F 1 "0.1uF" H 2015 1905 50  0000 L CNN
-F 2 "Capacitor_SMD:C_0603_1608Metric_Pad1.05x0.95mm_HandSolder" H 1938 1800 50  0001 C CNN
+F 2 "Capacitor_SMD:C_0603_1608Metric" H 1938 1800 50  0001 C CNN
 F 3 "~" H 1900 1950 50  0001 C CNN
 F 4 "1276-1000-1-ND" H 1900 1950 50  0001 C CNN "Digikey"
@@
 F 0 "C1" H 1165 1996 50  0000 L CNN
 F 1 "0.1uF" H 1165 1905 50  0000 L CNN
-F 2 "Capacitor_SMD:C_0603_1608Metric_Pad1.05x0.95mm_HandSolder" H 1088 1800 50  0001 C CNN
+F 2 "Capacitor_SMD:C_0603_1608Metric" H 1088 1800 50  0001 C CNN
 F 3 "~" H 1050 1950 50  0001 C CNN
 F 4 "1276-1000-1-ND" H 1050 1950 50  0001 C CNN "Digikey"
@@
 F 0 "C9" H 6615 1946 50  0000 L CNN
 F 1 "0.1uF" H 6615 1855 50  0000 L CNN
-F 2 "Capacitor_SMD:C_0603_1608Metric_Pad1.05x0.95mm_HandSolder" H 6538 1750 50  0001 C CNN
+F 2 "Capacitor_SMD:C_0603_1608Metric" H 6538 1750 50  0001 C CNN
 F 3 "~" H 6500 1900 50  0001 C CNN
 F 4 "1276-1000-1-ND" H 6500 1900 50  0001 C CNN "Digikey"
@@
 F 0 "C11" H 7015 1946 50  0000 L CNN
 F 1 "0.1uF" H 7015 1855 50  0000 L CNN
-F 2 "Capacitor_SMD:C_0603_1608Metric_Pad1.05x0.95mm_HandSolder" H 6938 1750 50  0001 C CNN
+F 2 "Capacitor_SMD:C_0603_1608Metric" H 6938 1750 50  0001 C CNN
 F 3 "~" H 6900 1900 50  0001 C CNN
 F 4 "1276-1000-1-ND" H 6900 1900 50  0001 C CNN "Digikey"
@@
 F 0 "C13" H 7415 1946 50  0000 L CNN
 F 1 "0.1uF" H 7415 1855 50  0000 L CNN
-F 2 "Capacitor_SMD:C_0603_1608Metric_Pad1.05x0.95mm_HandSolder" H 7338 1750 50  0001 C CNN
+F 2 "Capacitor_SMD:C_0603_1608Metric" H 7338 1750 50  0001 C CNN
 F 3 "~" H 7300 1900 50  0001 C CNN
 F 4 "1276-1000-1-ND" H 7300 1900 50  0001 C CNN "Digikey"
@@
 F 0 "C14" H 7815 1946 50  0000 L CNN
 F 1 "0.1uF" H 7815 1855 50  0000 L CNN
-F 2 "Capacitor_SMD:C_0603_1608Metric_Pad1.05x0.95mm_HandSolder" H 7738 1750 50  0001 C CNN
+F 2 "Capacitor_SMD:C_0603_1608Metric" H 7738 1750 50  0001 C CNN
 F 3 "~" H 7700 1900 50  0001 C CNN
 F 4 "1276-1000-1-ND" H 7700 1900 50  0001 C CNN "Digikey"
@@
 F 0 "C3" V 5100 850 50  0000 L CNN
 F 1 "4.7uF" V 4800 800 50  0000 L CNN
-F 2 "Capacitor_SMD:C_0603_1608Metric_Pad1.05x0.95mm_HandSolder" H 4988 750 50  0001 C CNN
+F 2 "Capacitor_SMD:C_0603_1608Metric" H 4988 750 50  0001 C CNN
 F 3 "~" H 4950 900 50  0001 C CNN
 F 4 "1276-6684-1-ND" H 4950 900 50  0001 C CNN "Digikey"
@@
 F 0 "C4" V 5100 1250 50  0000 L CNN
 F 1 "0.1uF" V 4800 1200 50  0000 L CNN
-F 2 "Capacitor_SMD:C_0603_1608Metric_Pad1.05x0.95mm_HandSolder" H 4988 1150 50  0001 C CNN
+F 2 "Capacitor_SMD:C_0603_1608Metric" H 4988 1150 50  0001 C CNN
 F 3 "~" H 4950 1300 50  0001 C CNN
 F 4 "1276-1000-1-ND" H 4950 1300 50  0001 C CNN "Digikey"
@@
 F 0 "C6" V 5100 1650 50  0000 L CNN
 F 1 "4.7uF" V 4800 1600 50  0000 L CNN
-F 2 "Capacitor_SMD:C_0603_1608Metric_Pad1.05x0.95mm_HandSolder" H 4988 1550 50  0001 C CNN
+F 2 "Capacitor_SMD:C_0603_1608Metric" H 4988 1550 50  0001 C CNN
 F 3 "~" H 4950 1700 50  0001 C CNN
 F 4 "1276-6684-1-ND" H 4950 1700 50  0001 C CNN "Digikey"
@@
 F 0 "C7" V 5100 2050 50  0000 L CNN
 F 1 "0.1uF" V 4800 2000 50  0000 L CNN
-F 2 "Capacitor_SMD:C_0603_1608Metric_Pad1.05x0.95mm_HandSolder" H 4988 1950 50  0001 C CNN
+F 2 "Capacitor_SMD:C_0603_1608Metric" H 4988 1950 50  0001 C CNN
 F 3 "~" H 4950 2100 50  0001 C CNN
 F 4 "1276-1000-1-ND" H 4950 2100 50  0001 C CNN "Digikey"
@@
 F 0 "C5" H 4165 2996 50  0000 L CNN
 F 1 "4.7uF" H 4165 2905 50  0000 L CNN
-F 2 "Capacitor_SMD:C_0603_1608Metric_Pad1.05x0.95mm_HandSolder" H 4088 2800 50  0001 C CNN
+F 2 "Capacitor_SMD:C_0603_1608Metric" H 4088 2800 50  0001 C CNN
 F 3 "~" H 4050 2950 50  0001 C CNN
 F 4 "1276-6684-1-ND" H 4050 2950 50  0001 C CNN "Digikey"
@@
 F 0 "C8" H 6615 1096 50  0000 L CNN
 F 1 "0.1uF" H 6615 1005 50  0000 L CNN
-F 2 "Capacitor_SMD:C_0603_1608Metric_Pad1.05x0.95mm_HandSolder" H 6538 900 50  0001 C CNN
+F 2 "Capacitor_SMD:C_0603_1608Metric" H 6538 900 50  0001 C CNN
 F 3 "~" H 6500 1050 50  0001 C CNN
 F 4 "1276-1000-1-ND" H 6500 1050 50  0001 C CNN "Digikey"
@@
 F 0 "C10" H 7015 1096 50  0000 L CNN
 F 1 "0.1uF" H 7015 1005 50  0000 L CNN
-F 2 "Capacitor_SMD:C_0603_1608Metric_Pad1.05x0.95mm_HandSolder" H 6938 900 50  0001 C CNN
+F 2 "Capacitor_SMD:C_0603_1608Metric" H 6938 900 50  0001 C CNN
 F 3 "~" H 6900 1050 50  0001 C CNN
 F 4 "1276-1000-1-ND" H 6900 1050 50  0001 C CNN "Digikey"
@@
 F 0 "C12" H 7415 1096 50  0000 L CNN
 F 1 "0.1uF" H 7415 1005 50  0000 L CNN
-F 2 "Capacitor_SMD:C_0603_1608Metric_Pad1.05x0.95mm_HandSolder" H 7338 900 50  0001 C CNN
+F 2 "Capacitor_SMD:C_0603_1608Metric" H 7338 900 50  0001 C CNN
 F 3 "~" H 7300 1050 50  0001 C CNN
 F 4 "1276-1000-1-ND" H 7300 1050 50  0001 C CNN "Digikey"
@@
 F 0 "C16" H 4265 6446 50  0000 L CNN
 F 1 "27pF" H 4265 6355 50  0000 L CNN
-F 2 "Capacitor_SMD:C_0603_1608Metric_Pad1.05x0.95mm_HandSolder" H 4188 6250 50  0001 C CNN
+F 2 "Capacitor_SMD:C_0603_1608Metric" H 4188 6250 50  0001 C CNN
 F 3 "~" H 4150 6400 50  0001 C CNN
 F 4 "1276-2247-1-ND" H 4150 6400 50  0001 C CNN "Digikey"
@@
 F 0 "C15" H 3765 6446 50  0000 L CNN
 F 1 "27pF" H 3765 6355 50  0000 L CNN
-F 2 "Capacitor_SMD:C_0603_1608Metric_Pad1.05x0.95mm_HandSolder" H 3688 6250 50  0001 C CNN
+F 2 "Capacitor_SMD:C_0603_1608Metric" H 3688 6250 50  0001 C CNN
 F 3 "~" H 3650 6400 50  0001 C CNN
 F 4 "1276-2247-1-ND" H 3650 6400 50  0001 C CNN "Digikey"
@@
 F 0 "R1" V 4250 3800 50  0000 C CNN
 F 1 "12k" V 4134 3800 50  0000 C CNN
-F 2 "Resistor_SMD:R_0603_1608Metric_Pad1.05x0.95mm_HandSolder" V 4180 3800 50  0001 C CNN
+F 2 "Resistor_SMD:R_0603_1608Metric" V 4180 3800 50  0001 C CNN
 F 3 "~" H 4250 3800 50  0001 C CNN
 	1    4250 3800
@@
 F 0 "R2" V 4250 4000 50  0000 C CNN
 F 1 "1k" V 4134 4000 50  0000 C CNN
-F 2 "Resistor_SMD:R_0603_1608Metric_Pad1.05x0.95mm_HandSolder" V 4180 4000 50  0001 C CNN
+F 2 "Resistor_SMD:R_0603_1608Metric" V 4180 4000 50  0001 C CNN
 F 3 "~" H 4250 4000 50  0001 C CNN
 	1    4250 4000
@@
 F 0 "R6" V 4300 4850 50  0000 C CNN
 F 1 "10k" V 4184 4850 50  0000 C CNN
-F 2 "Resistor_SMD:R_0603_1608Metric_Pad1.05x0.95mm_HandSolder" V 4230 4850 50  0001 C CNN
+F 2 "Resistor_SMD:R_0603_1608Metric" V 4230 4850 50  0001 C CNN
 F 3 "~" H 4300 4850 50  0001 C CNN
 	1    4300 4850
@@
 F 0 "R5" V 4100 4850 50  0000 C CNN
 F 1 "10k" V 3984 4850 50  0000 C CNN
-F 2 "Resistor_SMD:R_0603_1608Metric_Pad1.05x0.95mm_HandSolder" V 4030 4850 50  0001 C CNN
+F 2 "Resistor_SMD:R_0603_1608Metric" V 4030 4850 50  0001 C CNN
 F 3 "~" H 4100 4850 50  0001 C CNN
 	1    4100 4850
@@
 F 0 "R4" V 3900 4850 50  0000 C CNN
 F 1 "10k" V 3784 4850 50  0000 C CNN
-F 2 "Resistor_SMD:R_0603_1608Metric_Pad1.05x0.95mm_HandSolder" V 3830 4850 50  0001 C CNN
+F 2 "Resistor_SMD:R_0603_1608Metric" V 3830 4850 50  0001 C CNN
 F 3 "~" H 3900 4850 50  0001 C CNN
 	1    3900 4850
@@
 F 0 "R3" V 3350 5400 50  0000 C CNN
 F 1 "2.2k" V 3234 5400 50  0000 C CNN
-F 2 "Resistor_SMD:R_0603_1608Metric_Pad1.05x0.95mm_HandSolder" V 3280 5400 50  0001 C CNN
+F 2 "Resistor_SMD:R_0603_1608Metric" V 3280 5400 50  0001 C CNN
 F 3 "~" H 3350 5400 50  0001 C CNN
 	1    3350 5400
@@
 F 0 "C17" H 2415 1996 50  0000 L CNN
 F 1 "4.7uF" H 2415 1905 50  0000 L CNN
-F 2 "Capacitor_SMD:C_0603_1608Metric_Pad1.05x0.95mm_HandSolder" H 2338 1800 50  0001 C CNN
+F 2 "Capacitor_SMD:C_0603_1608Metric" H 2338 1800 50  0001 C CNN
 F 3 "~" H 2300 1950 50  0001 C CNN
 F 4 "1276-6684-1-ND" H 2300 1950 50  0001 C CNN "Digikey"

Commit message: Hmmm
Parts:
- renumbered C7 to C10, C8 to C11, C9 to C12, C10 to C13, C11 to C14, C12 to C15, C13 to C16, C14 to C17, C17 to C3, C15 to C4, C16 to C6, C3 to C7, C4 to C8, C6 to C9, R3 to R1, R4 to R2, R5 to R3, R1 to R4, R2 to R5, U2 to U1, U3 to U2, U1 to U3
